Commit message: Add Simple Examples and Logging Utilities (#28)

File: traj_opt/examples/2dof_spinner.urdf (robot description, URDF)
Before this commit: robot spinner, 4 links, 4 joints
Links:
- link finger_two: geometry collision sphere radius=.05; visual capsule length=0.9 radius=0.05
- link spinner: geometry collision capsule length=0.8 radius=0.25; visual capsule length=0.8 radius=0.25
Joints:
- joint theta_one: origin xyz=0 0 0 -> xyz=0 0 0 rpy=0 0.3 0; type continuous -> fixed

File: traj_opt/examples/2dof_spinner_capsule.urdf (robot description, URDF)
Before this commit: robot spinner, 4 links, 4 joints
Links:
- link finger_two: geometry collision capsule length=0.9 radius=0.05; visual capsule length=0.9 radius=0.05
- link spinner: geometry collision capsule length=0.8 radius=0.25; visual capsule length=0.8 radius=0.25
Joints:
- joint theta_one: origin xyz=0 0 0 -> xyz=0 0 0 rpy=0 0.3 0; type continuous -> fixed
