Commit message: Implement basic model predictive control in simulation (#61)
* simple multithreading example

* count to ten and simulate with u=0 at the same time

* refactor threads back into RunModelPredictiveControl function

* simple example of publishing LCM message from controller

* outline traj opt lcm interface tools

* send state measurements over lcm

* implement toy lcm controller

* multithreaded LCM controller working

* optimizer computes control torques, but doesn't update based on state

* fix controller output frequency

* update initial state for optimizer at each step

* acrobot MPC works at 100Hz (slowed simulation)

* acrobot MPC working in realtime

* better acrobot performance with low underactuation penalty

* use actuation matrix B to map optimizer results to control torques

* refactor examples to add MPC option

* pendulum mpc example

* spinner mpc working

* specify initial guess for mpc

* hopper mpc working

* refactor ControlWithStateFromLcm

* add profiling for MPC

* send nominal next state alongside torques as part of lcmt_traj_opt_u

* add low-level PD+ controller between MPC iterations

* add PD gains as yaml parameters

* try PD+ low level controller for hopper and spinner

* bounding velocity squared helps acrobot

* make maximum system energy a yaml parameter

* lint fixes

* put model files in separate directory

* add basic mini cheetah example

* copy cost parameters from hydroelastic iLQR paper

* shuffle forward at 1m/s

* minor cost function updates

* add torque limits: still not enough to prevent dramatic failure

* mildly improved hoopper example

* remove torque limits to fix acrobot example

* update hopper example parameters

* remove extra collision geometry on hopper for parity with traj_opt branch

* get rid of energy bound in low-level controller

* warm-start with full solve to convergence

* hopper parameter tuning for MPC

* update spinner markings

* convergence plots for dissertation draft

* realtime MPC with spinner

* cost tuning for a nice 2s trot

* 3 second demo gait

* better hopper and cheetah examples

* simple cost increasing problem isolation for mini cheetah

* isolate quaternion normalization as source of cost increase

* make normalize_quaternions a yaml parameter

* cleanup and lint fixes

* set params for spinner MPC

File: traj_opt/examples/models/spinner_friction.urdf (robot description, URDF)
Before this commit: robot spinner, 4 links, 4 joints
Links:
- link spinner: geometry collision sphere radius=0.25; visual cylinder length=0.5 radius=.04
